File: PCB/Project232/MCU.kicad_sch (KiCad schematic)
At the start: 28 parts, among them J1 BOOT MODE, J2 USB_B_Micro, J3 SW, SW1 RESET, U1 STM32F103C8Tx, U2 AMS1117-3.3

Commit message: update test board and docs
Parts:
- removed C12, C13, C14, C15: C, symbol Device:C
- removed R1: 100k, symbol Device:R_Small
- removed R3: R, symbol Device:R
- removed U2: AMS1117-3.3, Package_TO_SOT_SMD:SOT-223-3_TabPin2, symbol Regulator_Linear:AMS1117-3.3
- added R1: 150R, symbol Device:R_Small
- added R1: 100k, symbol Device:R_Small
- D1: value LED -> RED_LED
Connections:
- net +3V3: now also D1.2 (A)
- net BOOT0: now also R1.2
- net GND: no longer D1.1 (K)
- net DEBUG_LED: now reaches U1.2 (PC13)
- net DEBUG_LED: now also R1.1
- net at J1.2 (Pin_2): now also R1.1
- new net: D1.1 (K), R1.2
Other:
- removed sheet Sens
- removed sheet backup
- note added: "BOOT MODE"
- note added: "PLUG OUT THE BATTERY BEFORE USING USB PORT!"
- note added: "SPI CONNECTOR"
