File: PCB/Project232/Project232.kicad_sch (KiCad schematic)
At the start: 28 parts, among them J1 BOOT MODE, J2 USB_B_Micro, J3 SW, SW1 RESET, U1 STM32F103C8Tx, U2 AMS1117-3.3

Commit message: update test board and docs
Parts:
- removed C1, C16, C2, C3, C4: 100nF, symbol Device:C
- removed C10, C12, C13, C14, C15, C6, C7, C8, C9: C, symbol Device:C
- removed C11, C5: 4.7nF, symbol Device:C
- removed D1: LED, symbol Device:LED
- removed FB1: FerriteBead, symbol Device:FerriteBead
- removed HSE: 32MHz, symbol Device:Crystal_GND24
- removed J1: BOOT MODE, symbol Connector:Conn_01x03_Pin
- removed J2: USB_B_Micro, symbol Connector:USB_B_Micro
- removed J3: SW, symbol Connector:Conn_01x04_Pin
- removed R1: 100k, symbol Device:R_Small
- removed R2: R_Small, symbol Device:R_Small
- removed R3: R, symbol Device:R
- removed SW1: RESET, symbol Switch:SW_Push
- removed U1: STM32F103C8Tx, Package_QFP:LQFP-48_7x7mm_P0.5mm, symbol MCU_ST_STM32F1:STM32F103C8Tx
- removed U2: AMS1117-3.3, Package_TO_SOT_SMD:SOT-223-3_TabPin2, symbol Regulator_Linear:AMS1117-3.3
Connections:
- no-connect marks 2 -> 0
Other:
- added sheet MCU (MCU.kicad_sch)
- added sheet Power (Power.kicad_sch.kicad_sch)
- added sheet backup (backup.kicad_sch)

Commit message: Update PCB
Other:
- removed sheet backup
- sheet MCU ports: added BUCK_EN, CURR_IN, CURR_OUT, LOAD_CTR, PWM_PIN, VADC_IN, VADC_OUT; removed none
- sheet Sens ports: added BUCK_EN, CURR_IN, CURR_OUT, LOAD_CTR, PWM_PIN, VADC_IN, VADC_OUT; removed none
Changed lines of the file:
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@@
 (kicad_sch (version 20230121) (generator eeschema)
   (paper "A4")
-  (sheet (at 207.01 92.202) (size 36.322 48.006) (fields_autoplaced)
+  (wire (pts (xy 176.276 91.694) (xy 204.47 91.694))
+    (stroke (width 0) (type default))
+  )
+  (wire (pts (xy 176.276 115.316) (xy 204.47 115.316))
+    (stroke (width 0) (type default))
+  )
+  (wire (pts (xy 176.276 86.106) (xy 204.47 86.106))
+    (stroke (width 0) (type default))
+  )
+  (wire (pts (xy 176.276 111.76) (xy 204.47 111.76))
+    (stroke (width 0) (type default))
+  )
+  (wire (pts (xy 176.276 124.206) (xy 204.47 124.206))
+    (stroke (width 0) (type default))
+  )
+  (wire (pts (xy 176.276 97.028) (xy 204.47 97.028))
+    (stroke (width 0) (type default))
+  )
+  (wire (pts (xy 176.276 102.362) (xy 204.47 102.362))
+    (stroke (width 0) (type default))
+  )
+  (sheet (at 204.47 79.756) (size 36.322 48.006) (fields_autoplaced)
     (stroke (width 0.1524) (type solid))
     (fill (color 0 0 0 0.0000))
-    (property "Sheetname" "Sens" (at 207.01 91.4904 0)
+    (property "Sheetname" "Sens" (at 204.47 79.0444 0)
       (effects (font (size 1.27 1.27)) (justify left bottom))
     )
-    (property "Sheetfile" "Sens.kicad_sch" (at 207.01 140.7926 0)
+    (property "Sheetfile" "Sens.kicad_sch" (at 204.47 128.3466 0)
       (effects (font (size 1.27 1.27)) (justify left top))
+    )
+    (pin "CURR_IN" output (at 204.47 86.106 180)
+      (effects (font (size 1.27 1.27)) (justify left))
+    )
+    (pin "CURR_OUT" output (at 204.47 91.694 180)
+      (effects (font (size 1.27 1.27)) (justify left))
+    )
+    (pin "VADC_IN" output (at 204.47 97.028 180)
+      (effects (font (size 1.27 1.27)) (justify left))
+    )
+    (pin "PWM_PIN" input (at 204.47 111.76 180)
+      (effects (font (size 1.27 1.27)) (justify left))
+    )
+    (pin "BUCK_EN" input (at 204.47 115.316 180)
+      (effects (font (size 1.27 1.27)) (justify left))
+    )
+    (pin "LOAD_CTR" input (at 204.47 124.206 180)
+      (effects (font (size 1.27 1.27)) (justify left))
+    )
+    (pin "VADC_OUT" output (at 204.47 102.362 180)
+      (effects (font (size 1.27 1.27)) (justify left))
     )
     (instances
@@
     )
   )
-  (sheet (at 64.516 62.738) (size 27.94 34.036) (fields_autoplaced)
+  (sheet (at 67.31 91.186) (size 27.94 34.036) (fields_autoplaced)
     (stroke (width 0.1524) (type solid))
     (fill (color 0 0 0 0.0000))
-    (property "Sheetname" "Power" (at 64.516 62.0264 0)
+    (property "Sheetname" "Power" (at 67.31 90.4744 0)
       (effects (font (size 1.27 1.27)) (justify left bottom))
     )
-    (property "Sheetfile" "Power.kicad_sch.kicad_sch" (at 64.516 97.3586 0)
+    (property "Sheetfile" "Power.kicad_sch.kicad_sch" (at 67.31 125.8066 0)
       (effects (font (size 1.27 1.27)) (justify left top))
     )
@@
     )
   )
-  (sheet (at 249.682 16.764) (size 20.32 22.86) (fields_autoplaced)
+  (sheet (at 125.476 65.278) (size 50.8 81.026) (fields_autoplaced)
     (stroke (width 0.1524) (type solid))
     (fill (color 0 0 0 0.0000))
-    (property "Sheetname" "backup" (at 249.682 16.0524 0)
+    (property "Sheetname" "MCU" (at 125.476 64.5664 0)
       (effects (font (size 1.27 1.27)) (justify left bottom))
     )
-    (property "Sheetfile" "backup.kicad_sch" (at 249.682 40.2086 0)
+    (property "Sheetfile" "MCU.kicad_sch" (at 125.476 146.8886 0)
       (effects (font (size 1.27 1.27)) (justify left top))
     )
-    (property "Field2" "" (at 249.682 16.764 0)
-      (effects (font (size 1.27 1.27)) hide)
+    (pin "VADC_OUT" input (at 176.276 102.362 0)
+      (effects (font (size 1.27 1.27)) (justify right))
+    )
+    (pin "CURR_OUT" input (at 176.276 91.694 0)
+      (effects (font (size 1.27 1.27)) (justify right))
+    )
+    (pin "PWM_PIN" output (at 176.276 111.76 0)
+      (effects (font (size 1.27 1.27)) (justify right))
+    )
+    (pin "BUCK_EN" output (at 176.276 115.316 0)
+      (effects (font (size 1.27 1.27)) (justify right))
+    )
+    (pin "CURR_IN" input (at 176.276 86.106 0)
+      (effects (font (size 1.27 1.27)) (justify right))
+    )
+    (pin "VADC_IN" input (at 176.276 97.028 0)
+      (effects (font (size 1.27 1.27)) (justify right))
+    )
+    (pin "LOAD_CTR" output (at 176.276 124.206 0)
+      (effects (font (size 1.27 1.27)) (justify right))
     )
     (instances
-      (project "Project232"
-        (path "/b4ba9143-ff4b-4478-b064-00c745ce84f2" (page "3"))
-      )
-    )
-  )
-  (sheet (at 131.064 62.23) (size 50.8 81.026) (fields_autoplaced)
-    (stroke (width 0.1524) (type solid))
-    (fill (color 0 0 0 0.0000))
-    (property "Sheetname" "MCU" (at 131.064 61.5184 0)
-      (effects (font (size 1.27 1.27)) (justify left bottom))
-    )
-    (property "Sheetfile" "MCU.kicad_sch" (at 131.064 143.8406 0)
-      (effects (font (size 1.27 1.27)) (justify left top))
-    )
-    (instances
